File: SingleBMS/preautoroute.kicad_pcb (KiCad board)
At the start: 2 copper layers, 139.7 x 137.9 mm, 192 parts, among them J1 Conn_02x09_Top_Bottom, J2 Conn_02x09_Top_Bottom, J3 Conn_01x19, J4 Conn_01x19, J5 Conn_01x02, J6 Conn_01x08, J7 Conn_02x09_Top_Bottom, J8 Conn_01x02, Q1 2N7002, Q10 2N7002, Q11 2N7002, Q12 2N7002, Q13 2N7002, Q14 2N7002, Q15 2N7002, Q16 2N7002, Q2 2N7002, Q3 2N7002, Q4 2N7002, Q5 2N7002, Q6 2N7002, Q7 2N7002, Q8 2N7002, Q9 2N7002, U1 CD74HC4067M, U10 MCP23017_SP, U11 INA194, U12 MCP6004, U13 MCP6004, U14 MCP6004, U15 MCP6004, U16 PC817, U17 PC817, U18 PC817, U19 PC817, U2 PCF8574, U20 PC817, U21 PC817, U22 PC817, U23 PC817, U24 PC817, U25 PC817, U26 PC817, U27 PC817, U28 PC817, U29 PC817, U3 PCA9306, U30 PC817, U31 PC817, U4 ADS1115IDGS, U5 MCP6001-OT, U6 CD74HC4067M, U7 ESP32-DEVKITC-32D, U8 LM7805_TO220, U9 INA194

Commit message: Updated schematic with Vcc Globals, finished PCB layout, added screenshots
Connections:
- C1 pad 1: Vcc -> /Vcc
- C10 pad 2: Vcc -> /Vcc
- C11 pad 1: Vcc -> /Buffers16/Vcc
- C12 pad 1: Vcc -> /Buffers16/Vcc
- C13 pad 1: Vcc -> /Buffers16/Vcc
- C14 pad 1: Vcc -> /Buffers16/Vcc
- C2 pad 1: Vcc -> /Vcc
- C3 pad 1: Vcc -> /Vcc
- C4 pad 2: Vcc -> /Vcc
- C5 pad 2: Vcc -> /Vcc
- C6 pad 1: Vcc -> /Vcc
- C7 pad 2: Vcc -> /Vcc
- C9 pad 1: Vcc -> /Vcc
- J2 pad 18: Vcc -> /Vcc
- J3 pad 19: Vcc -> /Vcc
- J6 pad 1: Vcc -> /Vcc
- R1 pad 1: Vcc -> /Vcc
- R11 pad 1: Vcc -> /Vcc
- R6 pad 1: Vcc -> /Vcc
- U1 pad 24: Vcc -> /Vcc
- U10 pad 9: Vcc -> /Vcc
- U11 pad 5: Vcc -> /Vcc
- U12 pad 4: Vcc -> /Buffers16/Vcc
- U13 pad 4: Vcc -> /Buffers16/Vcc
- U14 pad 4: Vcc -> /Buffers16/Vcc
- U15 pad 4: Vcc -> /Buffers16/Vcc
- U2 pad 16: Vcc -> /Vcc
- U4 pad 8: Vcc -> /Vcc
- U5 pad 5: Vcc -> /Vcc
- U6 pad 24: Vcc -> /Vcc
- U7 pad 19: Vcc -> /Vcc
- U8 pad 3: Vcc -> /Vcc
- U9 pad 5: Vcc -> /Vcc
Routing:
- net Vcc: track 562.4 -> 0.00 mm
- net GND: track 548.7 -> 17.8 mm, vias 53 -> 0
- net /passiveBalance16/Bal9: track 112.9 -> 0.00 mm, vias 2 -> 0
- net /passiveBalance16/Bal8: track 105.0 -> 0.00 mm
- net /passiveBalance16/Bal11: track 100.5 -> 0.00 mm, vias 2 -> 0
- net /passiveBalance16/Bal7: track 98.7 -> 0.00 mm
- net /passiveBalance16/Bal10: track 96.7 -> 0.00 mm, vias 2 -> 0
- net /passiveBalance16/Bal12: track 95.8 -> 0.00 mm, vias 2 -> 0
- net /passiveBalance16/Bal6: track 93.6 -> 0.00 mm
- net /passiveBalance16/Bal13: track 88.7 -> 0.00 mm, vias 2 -> 0
- net /passiveBalance16/Bal5: track 87.9 -> 0.00 mm
- net /passiveBalance16/Bal14: track 83.5 -> 0.00 mm, vias 2 -> 0
- net /passiveBalance16/Bal4: track 81.5 -> 0.00 mm
- net /SDA: track 87.6 -> 6.34 mm, vias 3 -> 0
- net /passiveBalance16/Bal15: track 78.3 -> 0.00 mm, vias 2 -> 0
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- removed copper zone on F.Cu, net GND
Other:
- board outline removed
